File: hw/beacon.sch (KiCad schematic (older format))
At the start: 22 parts, among them J1 SPI_Prog_conn, Q1 Q_NMOS_DGS, Q2 Q_NMOS_DGS, Q3 Q_NMOS_DGS, U1 ATmega328-AU, U2 TSOP382xx

Commit message: Fixed hardware design errors
Missing connection between IR sensor and MCU
Wrong footprint for transistors
Parts:
- removed Q1, Q2, Q3: Q_NMOS_DGS, Package_TO_SOT_SMD:SOT-23_Handsoldering, symbol Device:Q_NMOS_DGS
- added Q1, Q2, Q3: Q_NMOS_GSD, Package_TO_SOT_SMD:SOT-23_Handsoldering, symbol Device:Q_NMOS_GSD
Connections:
- wire segments 69 -> 70
- no-connect marks 20 -> 19
Changed lines of the file:
@@
 EESchema Schematic File Version 4
+LIBS:beacon-cache
 EELAYER 26 0
 EELAYER END
@@
 $EndComp
 $Comp
-L Device:Q_NMOS_DGS Q1
-U 1 1 5B9B9A42
-P 7550 4750
-F 0 "Q1" H 7755 4796 50  0000 L CNN
-F 1 "Q_NMOS_DGS" H 7350 4950 50  0000 L CNN
-F 2 "Package_TO_SOT_SMD:SOT-23_Handsoldering" H 7750 4850 50  0001 C CNN
-F 3 "~" H 7550 4750 50  0001 C CNN
-	1    7550 4750
-	1    0    0    -1
-$EndComp
-$Comp
 L power:VCC #PWR0101
 U 1 1 5B9B9B69
@@
 LED_R_MCU_OUT
 $Comp
-L Device:Q_NMOS_DGS Q2
-U 1 1 5B9BE988
-P 8850 4750
-F 0 "Q2" H 9055 4796 50  0000 L CNN
-F 1 "Q_NMOS_DGS" H 8650 4950 50  0000 L CNN
-F 2 "Package_TO_SOT_SMD:SOT-23_Handsoldering" H 9050 4850 50  0001 C CNN
-F 3 "~" H 8850 4750 50  0001 C CNN
-	1    8850 4750
-	1    0    0    -1
-$EndComp
-$Comp
 L power:GND #PWR0108
 U 1 1 5B9BE98E
@@
 LED_G_MCU_OUT
 $Comp
-L Device:Q_NMOS_DGS Q3
-U 1 1 5B9BF051
-P 10200 4750
-F 0 "Q3" H 10405 4796 50  0000 L CNN
-F 1 "Q_NMOS_DGS" H 10000 4950 50  0000 L CNN
-F 2 "Package_TO_SOT_SMD:SOT-23_Handsoldering" H 10400 4850 50  0001 C CNN
-F 3 "~" H 10200 4750 50  0001 C CNN
-	1    10200 4750
-	1    0    0    -1
-$EndComp
-$Comp
 L power:GND #PWR0109
 U 1 1 5B9BF057
@@
 NoConn ~ 5350 4500
 NoConn ~ 5350 4400
-NoConn ~ 5350 4300
 NoConn ~ 5350 3700
 NoConn ~ 5350 3600
@@
 NoConn ~ 5350 2300
 NoConn ~ 4850 2000
+Wire Wire Line
+	5350 4300 6150 4300
+Text Label 6150 4300 0    50   ~ 0
+IR_MCU_IN
+$Comp
+L Device:Q_NMOS_GSD Q1
+U 1 1 5BF57757
+P 7550 4750
+F 0 "Q1" H 7755 4796 50  0000 L CNN
+F 1 "Q_NMOS_GSD" H 7755 4705 50  0000 L CNN
+F 2 "Package_TO_SOT_SMD:SOT-23_Handsoldering" H 7750 4850 50  0001 C CNN
+F 3 "~" H 7550 4750 50  0001 C CNN
+	1    7550 4750
+	1    0    0    -1
+$EndComp
+$Comp
+L Device:Q_NMOS_GSD Q2
+U 1 1 5BF57833
+P 8850 4750
+F 0 "Q2" H 9055 4796 50  0000 L CNN
+F 1 "Q_NMOS_GSD" H 9055 4705 50  0000 L CNN
+F 2 "Package_TO_SOT_SMD:SOT-23_Handsoldering" H 9050 4850 50  0001 C CNN
+F 3 "~" H 8850 4750 50  0001 C CNN
+	1    8850 4750
+	1    0    0    -1
+$EndComp
+$Comp
+L Device:Q_NMOS_GSD Q3
+U 1 1 5BF5796C
+P 10200 4750
+F 0 "Q3" H 10405 4796 50  0000 L CNN
+F 1 "Q_NMOS_GSD" H 10405 4705 50  0000 L CNN
+F 2 "Package_TO_SOT_SMD:SOT-23_Handsoldering" H 10400 4850 50  0001 C CNN
+F 3 "~" H 10200 4750 50  0001 C CNN
+	1    10200 4750
+	1    0    0    -1
+$EndComp
 $EndSCHEMATC
